Commit message: Add vehicle parameter synchronization system
- Created update_xacro_from_yaml.py to sync vehicle params from YAML to xacro files
- Updated noisy_odom_generator.py with covariance matrix updates
- Enhanced RunandGatherResults.py with dataset filtering and MPC type selection
- Integrated automatic xacro updates into runSimulator.sh and RunandGatherResults.py
- Fixed wheelbase discrepancy (2.84m -> 2.48m from vehicle_params.yaml)
- Added comprehensive documentation in VEHICLE_PARAMS_SYNC_README.md

🤖 Generated with [Claude Code](https://claude.com/claude-code)

Co-Authored-By: Claude <noreply@anthropic.com>

File: path_following_simulator/src/ackerman_ros_robot_gazebo_simulation/rbcar_common/rbcar_description/urdf/bases/rbcar_base.urdf.xacro (robot description, xacro)
@@ -34,8 +34,8 @@
   <link name="base_link">
     <inertial>
-      <mass value="125.0" />
-      <!-- <mass value="600.0" /> -->
+      <mass value="600" />
+      <!-- <mass value="600" /> -->
       <origin xyz="0 0 0" />
-      <inertia  ixx="1.391" ixy="0.0"  ixz="0.0"  iyy="6.853"  iyz="0.0"  izz="6.125" />
+      <inertia  ixx="216.5" ixy="0.0"  ixz="0.0"  iyy="843.9"  iyz="0.0"  izz="771.4" />
     </inertial>
     <visual>

File: path_following_simulator/src/ackerman_ros_robot_gazebo_simulation/rbcar_common/rbcar_description/urdf/wheels/suspension_wheel.urdf.xacro (robot description, xacro)
@@ -22,4 +22,5 @@
   <!-- Degree-to-radian conversions -->
   <xacro:property name="degrees_45" value="0.785398163"/>
+  <xacro:property name="steer_limit" value="0.444"/>
   <xacro:property name="degrees_90" value="1.57079633"/>
   <xacro:property name="degrees_180" value="3.14159265"/>
@@ -43,5 +44,5 @@
        measured in rad/s. -->
   <xacro:property name="servo_stall_torque" value="50"/>  <!-- check -->
-  <xacro:property name="servo_no_load_speed" value="25"/> <!-- check -->
+  <xacro:property name="servo_no_load_speed" value="0.14"/> <!-- check -->
   <!-- Inertia of a thick-walled cylindrical tube with open ends. Height is
        measured along the z axis, which is the tube's axis. inner_rad and
@@ -186,5 +187,5 @@
       <child link="${lr_prefix}_${fr_prefix}_axle_carrier"/>
       <axis xyz="0 0 1"/>
-      <limit lower="${-degrees_45}" upper="${degrees_45}"
+      <limit lower="-${steer_limit}" upper="${steer_limit}"
              effort="${servo_stall_torque}" velocity="${servo_no_load_speed}"/>
     </joint>
