Commit message: chore: Update simulation configuration and scripts

File: path_following_simulator/src/ackerman_ros_robot_gazebo_simulation/rbcar_common/rbcar_description/urdf/bases/rbcar_base.urdf.xacro (robot description, xacro)
@@ -11,5 +11,5 @@
     <link name="base_footprint">
       <visual>
-          <origin xyz="1.24 0 0" rpy="0 0 0" />
+          <origin xyz="${wheelbase/2} 0 0" rpy="0 0 0" />
           <geometry>
              <box size="0.001 0.001 0.001" />
@@ -26,5 +26,5 @@
     </link>
     <joint name="base_footprint_joint" type="fixed">
-      <origin xyz="1.24 0 ${clearance}" rpy="0 0 0" />  <!-- height is the clearance -->
+      <origin xyz="${wheelbase/2} 0 ${clearance}" rpy="0 0 0" />  <!-- height is the clearance -->
       <parent link="base_footprint"/>
       <child link="base_link" />
